Commit message: Add cultivator implement

File: romea_implement_description/urdf/hitch_implement.xacro (robot description, xacro)
@@ -2,5 +2,5 @@
 <robot xmlns:xacro="http://wiki.ros.org/xacro" name="hitch_implement">
    <xacro:macro name="hitch_implement"
-      params="prefix mode name model xyz rpy parent_link controller_manager_config_yaml_file ros2_control_config_urdf_file ros_prefix ros_distro">
+      params="prefix mode name xyz rpy parent_link controller_manager_config_yaml_file ros2_control_config_urdf_file ros_prefix ros_distro *geometry">
       <xacro:property
          name="hitch_prefix"
@@ -9,10 +9,4 @@
          name="parent_link_name"
          value="${prefix}${parent_link}" />
-      <xacro:property
-         name="hitch_type"
-         value="hitch${model}" />
-      <!-- <xacro:property
-         name="visual_params_file"
-         value="$(find hitch_description)/config/${hitch_type}/visual_parameters.yaml" /> -->
       <!-- implement -->
       <xacro:include filename="$(find romea_implement_description)/urdf/common.xacro" />
@@ -28,21 +22,17 @@
       <link name="${hitch_prefix}_hitch_link">
          <visual>
-            <geometry>
-               <box size="1.0 2.0 0.5" />
-            </geometry>
-            <origin xyz="0 0 -1." rpy="0 -${pi/2} 0 " />
+            <xacro:insert_block name="geometry" />
+            <origin xyz="0 0 0" rpy="0 -${pi/2} 0 " />
          </visual>
          <collision>
-            <geometry>
-               <box size="1.0 2.0 0.5" />
-            </geometry>
-            <origin xyz="0 0 -1." rpy="0 -${pi/2} 0 " />
+            <xacro:insert_block name="geometry" />
+            <origin xyz="0 0 0" rpy="0 -${pi/2} 0 " />
          </collision>
-         <xacro:inertial_dummy />
+         <xacro:inertial_cuboid mass="100." x="1." y="2." z="0.5" />
       </link>
       <joint name="${hitch_prefix}_hitch_joint" type="prismatic">
          <parent link="${hitch_prefix}_link" />
          <child link="${hitch_prefix}_hitch_link" />
-         <limit effort="1000.0" lower="0" upper="0.5" velocity="0.5" />
+         <limit effort="1000.0" lower="0" upper="1.0" velocity="0.5" />
          <origin rpy="0 ${pi/2} 0" xyz="0 0 0" />
       </joint>

Commit message: Use position pid for implement control

File: romea_implement_description/urdf/hitch_implement.xacro (robot description, xacro)
@@ -17,6 +17,6 @@
       <joint name="${hitch_prefix}_joint" type="fixed">
          <origin xyz="${xyz}" rpy="${rpy}" />
+         <parent link="${parent_link_name}" />
          <child link="${hitch_prefix}_link" />
-         <parent link="${parent_link_name}" />
       </joint>
       <link name="${hitch_prefix}_hitch_link">
@@ -32,8 +32,9 @@
       </link>
       <joint name="${hitch_prefix}_hitch_joint" type="prismatic">
+         <origin rpy="0 ${pi/2} 0" xyz="0 0 0" />
          <parent link="${hitch_prefix}_link" />
          <child link="${hitch_prefix}_hitch_link" />
-         <limit effort="1000.0" lower="0" upper="1.0" velocity="0.5" />
-         <origin rpy="0 ${pi/2} 0" xyz="0 0 0" />
+         <dynamics damping="2000.0" friction="40." />
+         <limit effort="10000.0" lower="0" upper="1.0" velocity="0.1" />
       </joint>
       <ros2_control name="${hitch_prefix}" type="system">
@@ -44,8 +45,14 @@
          </xacro:if>
          <joint name="${hitch_prefix}_hitch_joint">
-            <command_interface name="position" />
-            <command_interface name="velocity" />
+            <param name="pos_kp">100000</param>
+            <param name="pos_ki">10.</param>
+            <param name="pos_kd">0</param>
+            <param name="pos_max_integral_error">10000</param>
+            <command_interface name="effort" />
+            <!-- <command_interface name="position" /> -->
+            <command_interface name="position_pid" />
             <state_interface name="position" />
             <state_interface name="velocity" />
+            <state_interface name="effort" />
          </joint>
       </ros2_control>

Commit message: Introduce offset between visual and collision

File: romea_implement_description/urdf/hitch_implement.xacro (robot description, xacro)
@@ -27,5 +27,5 @@
          <collision>
             <xacro:insert_block name="geometry" />
-            <origin xyz="0 0 0" rpy="0 -${pi/2} 0 " />
+            <origin xyz="-0.05 0 0" rpy="0 -${pi/2} 0 " />
          </collision>
          <xacro:inertial_cuboid mass="100." x="1." y="2." z="0.5" />

Commit message: add collision bitmask in URDF

File: romea_implement_description/urdf/hitch_implement.xacro (robot description, xacro)
@@ -27,5 +27,5 @@
          <collision>
             <xacro:insert_block name="geometry" />
-            <origin xyz="-0.05 0 0" rpy="0 -${pi/2} 0 " />
+            <origin xyz="0 0 0" rpy="0 -${pi/2} 0 " />
          </collision>
          <xacro:inertial_cuboid mass="100." x="1." y="2." z="0.5" />
@@ -67,4 +67,15 @@
             </plugin>
          </gazebo>
+         <gazebo reference="${hitch_prefix}_hitch_link">
+            <collision>
+               <surface>
+                  <contact>
+                     <!-- bitmask: stems(4), weeds(3), crops(2), elements(1), ground(0) -->
+                     <!-- in this case: no contact with weeds and ground -->
+                     <collide_bitmask>0x16</collide_bitmask>
+                  </contact>
+               </surface>
+            </collision>
+         </gazebo>
       </xacro:if>
    </xacro:macro>

Commit message: Modify implement macro

File: romea_implement_description/urdf/hitch_implement.xacro (robot description, xacro)
@@ -2,5 +2,5 @@
 <robot xmlns:xacro="http://wiki.ros.org/xacro" name="hitch_implement">
    <xacro:macro name="hitch_implement"
-      params="prefix mode name xyz rpy parent_link controller_manager_config_yaml_file ros2_control_config_urdf_file ros_prefix ros_distro *visual_geometry *collision_geometry">
+      params="prefix mode name xyz rpy parent_link controller_manager_config_yaml_file ros2_control_config_urdf_file ros_prefix ros_distro *visual *collision">
       <xacro:property
          name="hitch_prefix"
@@ -21,12 +21,6 @@
       </joint>
       <link name="${hitch_prefix}_hitch_link">
-         <visual>
-            <xacro:insert_block name="visual_geometry" />
-            <origin xyz="0 0 0" rpy="0 -${pi/2} 0 " />
-         </visual>
-         <collision>
-            <xacro:insert_block name="collision_geometry" />
-            <origin xyz="0 0 0" rpy="0 -${pi/2} 0 " />
-         </collision>
+         <xacro:insert_block name="visual"/>
+         <xacro:insert_block name="collision"/>
          <xacro:inertial_cuboid mass="100." x="1." y="2." z="0.5" />
       </link>
